Commit message: URDFファイル内LiDARとカメラの位置関係修正

File: urdf/mirs.urdf (robot description, URDF)
Before this commit: robot cleaning_robot, 6 links, 5 joints
Links:
- removed link camera_link
- removed link laser_frame
- added link camera; visual box size=0.02 0.05 0.02
- added link laser; visual cylinder length=0.04 radius=0.035
Joints:
- joint camera_joint: child camera_link -> camera; origin xyz=0.20 0 0.30 rpy=0 0 0 -> xyz=0.15 0 0.3 rpy=-1.5707 0 -1.5707; parent base_footprint -> base_link
- joint lidar_joint: child laser_frame -> laser; origin xyz=0 0 0.3 rpy=3.14159 0 0 -> xyz=0 0 0.3 rpy=0 0 0; parent base_footprint -> base_link

Commit message: urdfファイル内ロボットサイズ定義変更

File: urdf/mirs.urdf (robot description, URDF)
Before this commit: robot cleaning_robot, 6 links, 5 joints
Links:
- link base_link: geometry collision box size=0.50 0.50 0.20; visual box size=0.50 0.50 0.20

Commit message: LiDAR/カメラの位置を変更

File: urdf/mirs.urdf (robot description, URDF)
Before this commit: robot cleaning_robot, 6 links, 5 joints
Joints:
- joint camera_joint: origin xyz=0.15 0 0.3 rpy=-1.5707 0 -1.5707 -> xyz=0.27 0 0.15 rpy=0 0 0
- joint lidar_joint: origin xyz=0 0 0.3 rpy=0 0 0 -> xyz=0 0 0.105 rpy=3.14159 0 0

Commit message: URDFファイルのホイール径を修正

File: urdf/mirs.urdf (robot description, URDF)
Before this commit: robot cleaning_robot, 6 links, 5 joints
Links:
- link left_wheel: geometry visual cylinder length=0.05 radius=0.0391
- link right_wheel: geometry visual cylinder length=0.05 radius=0.0391
Joints:
- joint base_joint: origin xyz=0 0 0.10 rpy=0 0 0 -> xyz=0 0 0.0391 rpy=0 0 0
- joint camera_joint: origin xyz=0.27 0 0.15 rpy=0 0 0 -> xyz=0.15 0 0.3 rpy=-1.5707 0 -1.5707
- joint left_wheel_joint: origin xyz=0 0.225 0 rpy=0 0 0 -> xyz=0 0.212 0 rpy=0 0 0
- joint right_wheel_joint: origin xyz=0 -0.225 0 rpy=0 0 0 -> xyz=0 -0.212 0 rpy=0 0 0
